File: 40Left.kicad_pcb (KiCad board)
At the start: 2 copper layers, 340 x 80.5 mm, 123 parts, among them SW1 SW_PUSH, SW10 SW_PUSH, SW11 SW_PUSH, SW12 SW_PUSH, SW13 SW_PUSH, SW14 SW_PUSH, SW15 SW_PUSH, SW16 SW_PUSH, SW17 SW_PUSH, SW18 SW_PUSH, SW19 SW_PUSH, SW2 SW_PUSH, SW20 SW_PUSH, SW21 SW_PUSH, SW22 SW_PUSH, SW23 SW_PUSH, SW24 SW_PUSH, SW25 SW_PUSH, SW26 SW_PUSH, SW27 SW_PUSH, SW28 SW_PUSH, SW29 SW_PUSH, SW3 SW_PUSH, SW30 SW_PUSH, SW31 SW_PUSH, SW32 SW_PUSH, SW33 SW_PUSH, SW34 SW_PUSH, SW35 SW_PUSH, SW37 SW_PUSH, SW38 SW_PUSH, SW39 SW_PUSH, SW4 SW_PUSH, SW40 SW_PUSH, SW41 SW_PUSH, SW42 SW_PUSH, SW43 SW_PUSH, SW45 SW_PUSH, SW46 SW_PUSH, SW47 SW_PUSH, SW48 SW_PUSH, SW49 SW_PUSH, SW5 SW_PUSH, SW50 SW_PUSH, SW51 SW_PUSH, SW52 SW_PUSH, SW53 SW_PUSH, SW54 SW_PUSH, SW55 SW_PUSH, SW57 SW_PUSH, SW58 SW_PUSH, SW59 SW_PUSH, SW6 SW_PUSH, SW60 SW_PUSH, SW61 SW_PUSH, SW62 SW_PUSH, SW63 SW_PUSH, SW64 SW_PUSH, SW7 SW_PUSH, SW8 SW_PUSH, SW9 SW_PUSH, U1 ProMicro

Commit message: updated the footprint.
Parts:
- D1, D10, D11, D12, D13, D14, D15, D16, D17, D18, D19, D2, D20, D21, D22, D23, D24, D25, D26, D27, D28, D29, D3, D30, D31, D32, D33, D34, D35, D37, D38, D39, D4, D40, D41, D42, D43, D45, D46, D47, D48, D49, D5, D50, D51, D52, D53, D54, D55, D57, D58, D59, D6, D60, D61, D62, D63, D64, D7, D8, D9: footprint Keebio-Parts:Diode -> footprints:diode
- SW1, SW10, SW11, SW12, SW13, SW14, SW15, SW16, SW17, SW2, SW21, SW22, SW23, SW24, SW25, SW26, SW27, SW29, SW3, SW30, SW31, SW33, SW34, SW35, SW37, SW38, SW39, SW4, SW40, SW41, SW42, SW43, SW45, SW46, SW47, SW49, SW5, SW50, SW51, SW52, SW53, SW54, SW55, SW57, SW58, SW59, SW6, SW60, SW63, SW7, SW8, SW9: footprint Keebio-Parts:MX_PCB_100H -> footprints:100-minimal
- SW18, SW20, SW28, SW64: footprint Keebio-Parts:MX_PCB_125H -> footprints:125-minimal
- SW19, SW61: footprint Keebio-Parts:MX_PCB_175H -> footprints:175-minimal
- SW32: footprint Keebio-Parts:MX_PCB_225H -> footprints:225-minimal
- SW48: footprint Keebio-Parts:MX_PCB_275H -> footprints:275-minimal
- SW62: footprint Keebio-Parts:MX_PCB_150H -> footprints:150-minimal
- U1: footprint promicro:ProMicro -> footprints:promicro
- moved U1 2.50 mm to (107.3, 38.5)
- turned D1 to 0 degrees
- turned D10 to 0 degrees
- turned D11 to 0 degrees
- turned D12 to 0 degrees
- turned D13 to 0 degrees
- turned D14 to 0 degrees
- turned D15 to 0 degrees
- turned D16 to 0 degrees
- turned D17 to 0 degrees
- turned D18 to 0 degrees
- turned D19 to 0 degrees
- turned D2 to 0 degrees
- turned D20 to 0 degrees
- turned D21 to 0 degrees
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Connections:
- SW1 pad 1: Net-(D1-Pad2) -> C01
- SW1 pad 2: C01 -> Net-(D1-Pad2)
- SW10 pad 1: Net-(D10-Pad2) -> C23
- SW10 pad 2: C23 -> Net-(D10-Pad2)
- SW11 pad 1: Net-(D11-Pad2) -> C23
- SW11 pad 2: C23 -> Net-(D11-Pad2)
- SW12 pad 1: Net-(D12-Pad2) -> C23
- SW12 pad 2: C23 -> Net-(D12-Pad2)
- SW13 pad 1: Net-(D13-Pad2) -> C23
- SW13 pad 2: C23 -> Net-(D13-Pad2)
- SW14 pad 1: Net-(D14-Pad2) -> C23
- SW14 pad 2: C23 -> Net-(D14-Pad2)
- SW15 pad 1: Net-(D15-Pad2) -> C23
- SW15 pad 2: C23 -> Net-(D15-Pad2)
- SW16 pad 1: Net-(D16-Pad2) -> C23
- SW16 pad 2: C23 -> Net-(D16-Pad2)
- SW17 pad 1: Net-(D17-Pad2) -> C45
- SW17 pad 2: C45 -> Net-(D17-Pad2)
- SW18 pad 1: Net-(D18-Pad2) -> C45
- SW18 pad 2: C45 -> Net-(D18-Pad2)
- SW19 pad 1: Net-(D19-Pad2) -> C45
- SW19 pad 2: C45 -> Net-(D19-Pad2)
- SW2 pad 1: Net-(D2-Pad2) -> C01
- SW2 pad 2: C01 -> Net-(D2-Pad2)
- SW20 pad 1: Net-(D20-Pad2) -> C45
- SW20 pad 2: C45 -> Net-(D20-Pad2)
- SW21 pad 1: Net-(D21-Pad2) -> C45
- SW21 pad 2: C45 -> Net-(D21-Pad2)
- SW22 pad 1: Net-(D22-Pad2) -> C45
- SW22 pad 2: C45 -> Net-(D22-Pad2)
- SW23 pad 1: Net-(D23-Pad2) -> C45
- SW23 pad 2: C45 -> Net-(D23-Pad2)
- SW24 pad 1: Net-(D24-Pad2) -> C45
- SW24 pad 2: C45 -> Net-(D24-Pad2)
- SW25 pad 1: Net-(D25-Pad2) -> C67
- SW25 pad 2: C67 -> Net-(D25-Pad2)
- SW26 pad 1: Net-(D26-Pad2) -> C67
- SW26 pad 2: C67 -> Net-(D26-Pad2)
- SW27 pad 1: Net-(D27-Pad2) -> C67
- SW27 pad 2: C67 -> Net-(D27-Pad2)
- SW28 pad 1: Net-(D28-Pad2) -> C67
- SW28 pad 2: C67 -> Net-(D28-Pad2)
- SW29 pad 1: Net-(D29-Pad2) -> C67
- SW29 pad 2: C67 -> Net-(D29-Pad2)
- SW3 pad 1: Net-(D3-Pad2) -> C01
- SW3 pad 2: C01 -> Net-(D3-Pad2)
- SW30 pad 1: Net-(D30-Pad2) -> C67
- SW30 pad 2: C67 -> Net-(D30-Pad2)
- SW31 pad 1: Net-(D31-Pad2) -> C67
- SW31 pad 2: C67 -> Net-(D31-Pad2)
- SW33 pad 1: Net-(D33-Pad2) -> C89
- SW33 pad 2: C89 -> Net-(D33-Pad2)
- SW34 pad 1: Net-(D34-Pad2) -> C89
- SW34 pad 2: C89 -> Net-(D34-Pad2)
- SW35 pad 1: Net-(D35-Pad2) -> C89
- SW35 pad 2: C89 -> Net-(D35-Pad2)
- SW37 pad 1: Net-(D37-Pad2) -> C89
- SW37 pad 2: C89 -> Net-(D37-Pad2)
- SW38 pad 1: Net-(D38-Pad2) -> C89
- SW38 pad 2: C89 -> Net-(D38-Pad2)
- SW39 pad 1: Net-(D39-Pad2) -> C89
- SW39 pad 2: C89 -> Net-(D39-Pad2)
- SW4 pad 1: Net-(D4-Pad2) -> C01
- SW4 pad 2: C01 -> Net-(D4-Pad2)
- SW40 pad 1: Net-(D40-Pad2) -> C89
- SW40 pad 2: C89 -> Net-(D40-Pad2)
- SW41 pad 1: Net-(D41-Pad2) -> CAB
- SW41 pad 2: CAB -> Net-(D41-Pad2)
- SW42 pad 1: Net-(D42-Pad2) -> CAB
- SW42 pad 2: CAB -> Net-(D42-Pad2)
- SW43 pad 1: Net-(D43-Pad2) -> CAB
- SW43 pad 2: CAB -> Net-(D43-Pad2)
- SW45 pad 1: Net-(D45-Pad2) -> CAB
- SW45 pad 2: CAB -> Net-(D45-Pad2)
- SW46 pad 1: Net-(D46-Pad2) -> CAB
- SW46 pad 2: CAB -> Net-(D46-Pad2)
- SW47 pad 1: Net-(D47-Pad2) -> CAB
- SW47 pad 2: CAB -> Net-(D47-Pad2)
- SW49 pad 1: Net-(D49-Pad2) -> CCD
- SW49 pad 2: CCD -> Net-(D49-Pad2)
- SW5 pad 1: Net-(D5-Pad2) -> C01
- SW5 pad 2: C01 -> Net-(D5-Pad2)
- SW50 pad 1: Net-(D50-Pad2) -> CCD
- SW50 pad 2: CCD -> Net-(D50-Pad2)
- SW51 pad 1: Net-(D51-Pad2) -> CCD
- SW51 pad 2: CCD -> Net-(D51-Pad2)
- SW52 pad 1: Net-(D52-Pad2) -> CCD
- SW52 pad 2: CCD -> Net-(D52-Pad2)
- SW53 pad 1: Net-(D53-Pad2) -> CCD
- SW53 pad 2: CCD -> Net-(D53-Pad2)
- SW54 pad 1: Net-(D54-Pad2) -> CCD
- SW54 pad 2: CCD -> Net-(D54-Pad2)
- SW55 pad 1: Net-(D55-Pad2) -> CCD
- SW55 pad 2: CCD -> Net-(D55-Pad2)
- SW57 pad 1: Net-(D57-Pad2) -> CEF
- SW57 pad 2: CEF -> Net-(D57-Pad2)
- SW58 pad 1: Net-(D58-Pad2) -> CEF
- SW58 pad 2: CEF -> Net-(D58-Pad2)
- SW59 pad 1: Net-(D59-Pad2) -> CEF
- SW59 pad 2: CEF -> Net-(D59-Pad2)
- SW6 pad 1: Net-(D6-Pad2) -> C01
- SW6 pad 2: C01 -> Net-(D6-Pad2)
- SW60 pad 1: Net-(D60-Pad2) -> CEF
- SW60 pad 2: CEF -> Net-(D60-Pad2)
- SW61 pad 1: Net-(D61-Pad2) -> CEF
- SW61 pad 2: CEF -> Net-(D61-Pad2)
- SW62 pad 1: Net-(D62-Pad2) -> CEF
- SW62 pad 2: CEF -> Net-(D62-Pad2)
- SW63 pad 1: Net-(D63-Pad2) -> CEF
- SW63 pad 2: CEF -> Net-(D63-Pad2)
- SW64 pad 1: Net-(D64-Pad2) -> CEF
- SW64 pad 2: CEF -> Net-(D64-Pad2)
- SW7 pad 1: Net-(D7-Pad2) -> C01
- SW7 pad 2: C01 -> Net-(D7-Pad2)
- SW8 pad 1: Net-(D8-Pad2) -> C01
- SW8 pad 2: C01 -> Net-(D8-Pad2)
- SW9 pad 1: Net-(D9-Pad2) -> C23
- SW9 pad 2: C23 -> Net-(D9-Pad2)
- U1 pad 19: Net-(U1-Pad19) -> (no net)
- U1 pad 20: Net-(U1-Pad20) -> (no net)
- U1 pad 21: Net-(U1-Pad21) -> (no net)
- U1 pad 22: Net-(U1-Pad22) -> (no net)
- U1 pad 23: Net-(U1-Pad23) -> (no net)
- U1 pad 24: Net-(U1-Pad24) -> (no net)
- U1 pad 3: Net-(U1-Pad3) -> (no net)
- U1 pad 4: Net-(U1-Pad4) -> (no net)
Routing:
- net R1B: track 310.8 -> 388.6 mm
- net C67: track 223.3 -> 257.0 mm
- net CAB: track 282.6 -> 308.7 mm
- net C45: track 181.7 -> 203.4 mm
- net C89: track 240.1 -> 261.7 mm
- net CCD: track 325.2 -> 340.3 mm
- net CEF: track 391.0 -> 403.1 mm
- net R0B: track 312.2 -> 317.3 mm
- net R1A: track 298.3 -> 302.0 mm, vias 1 -> 0
- net R0A: track 302.9 -> 306.5 mm
- net R2B: track 337.7 -> 335.1 mm
- net R2A: track 333.3 -> 330.7 mm
- net R3B: track 360.6 -> 362.9 mm
- net Net-(D32-Pad2): track 17.0 -> 18.2 mm
- net Net-(D48-Pad2): track 17.4 -> 18.6 mm
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- added copper zone on B.Cu, net (none)
- added copper zone on F.Cu, net (none)
Other:
- board size 340 x 80.5 mm -> 340 x 77 mm
- board text added: "THIS KEYBOARD IS DEDICATED TO THE BRAVE MUJAHIDEEN FIGHTERS OF AFGHANISTAN"

Commit message: shorter.
Parts:
- SW19, SW61: footprint footprints:175-minimal -> footprints:150-minimal
- SW48: footprint footprints:275-minimal -> footprints:225-minimal
- SW52: footprint footprints:100-minimal -> footprints:125-minimal
- SW62: footprint footprints:150-minimal -> footprints:125-minimal
- moved D13 23.5 mm to (118.5, 32.0)
- moved D1 21.0 mm to (59.0, 30.0)
- moved D11 21.0 mm to (97.0, 68.0)
- moved D12 21.0 mm to (97.0, 87.0)
- moved D15 21.0 mm to (116.0, 70.0)
- moved D16 21.0 mm to (116.0, 89.0)
- moved D2 21.0 mm to (59.0, 49.0)
- moved D3 21.0 mm to (59.0, 68.0)
- moved D4 21.0 mm to (59.0, 87.0)
- moved D5 21.0 mm to (78.0, 32.0)
- moved D6 21.0 mm to (78.0, 51.0)
- moved D7 21.0 mm to (78.0, 70.0)
- moved D8 21.0 mm to (78.0, 89.0)
- moved D9 21.0 mm to (97.0, 30.0)
- moved SW1 21.0 mm to (51.0, 30.0)
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Routing:
- net R1B: track 388.6 -> 283.5 mm
- net CEF: track 403.1 -> 363.3 mm
- net CCD: track 340.3 -> 307.5 mm
- net R2A: track 330.7 -> 301.8 mm, vias 1 -> 0
- net CAB: track 308.7 -> 281.6 mm
- net R1A: track 302.0 -> 275.9 mm
- net R3A: track 353.8 -> 328.6 mm, vias 1 -> 0
- net C89: track 261.7 -> 239.1 mm
- net R0A: track 306.5 -> 285.5 mm
- net C45: track 203.4 -> 182.7 mm
- net R0B: track 317.3 -> 296.9 mm
- net C01: track 189.6 -> 169.3 mm
- net R2B: track 335.1 -> 355.4 mm
- net C23: track 152.3 -> 134.6 mm
- net C67: track 257.0 -> 239.6 mm
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Other:
- board size 340 x 77 mm -> 314.2 x 77 mm
