File: 40Left.sch (KiCad schematic (older format))
At the start: 123 parts, among them SW1 SW_PUSH, SW10 SW_PUSH, SW11 SW_PUSH, SW12 SW_PUSH, SW13 SW_PUSH, SW14 SW_PUSH, SW15 SW_PUSH, SW16 SW_PUSH, SW17 SW_PUSH, SW18 SW_PUSH, SW19 SW_PUSH, SW2 SW_PUSH, SW20 SW_PUSH, SW21 SW_PUSH, SW22 SW_PUSH, SW23 SW_PUSH, SW24 SW_PUSH, SW25 SW_PUSH, SW26 SW_PUSH, SW27 SW_PUSH, SW28 SW_PUSH, SW29 SW_PUSH, SW3 SW_PUSH, SW30 SW_PUSH, SW31 SW_PUSH, SW32 SW_PUSH, SW33 SW_PUSH, SW34 SW_PUSH, SW35 SW_PUSH, SW37 SW_PUSH, SW38 SW_PUSH, SW39 SW_PUSH, SW4 SW_PUSH, SW40 SW_PUSH, SW41 SW_PUSH, SW42 SW_PUSH, SW43 SW_PUSH, SW45 SW_PUSH, SW46 SW_PUSH, SW47 SW_PUSH, SW48 SW_PUSH, SW49 SW_PUSH, SW5 SW_PUSH, SW50 SW_PUSH, SW51 SW_PUSH, SW52 SW_PUSH, SW53 SW_PUSH, SW54 SW_PUSH, SW55 SW_PUSH, SW57 SW_PUSH, SW58 SW_PUSH, SW59 SW_PUSH, SW6 SW_PUSH, SW60 SW_PUSH, SW61 SW_PUSH, SW62 SW_PUSH, SW63 SW_PUSH, SW64 SW_PUSH, SW7 SW_PUSH, SW8 SW_PUSH, SW9 SW_PUSH, U1 ProMicro

Commit message: updated the footprint.
Parts:
- D1, D10, D11, D12, D13, D14, D15, D16, D17, D18, D19, D2, D20, D21, D22, D23, D24, D25, D26, D27, D28, D29, D3, D30, D31, D32, D33, D34, D35, D37, D38, D39, D4, D40, D41, D42, D43, D45, D46, D47, D48, D49, D5, D50, D51, D52, D53, D54, D55, D57, D58, D59, D6, D60, D61, D62, D63, D64, D7, D8, D9: footprint Keebio-Parts:Diode -> footprints:diode; symbol keyboard_parts:D -> rick-kicad-lib:diode
- SW1, SW10, SW11, SW12, SW13, SW14, SW15, SW16, SW17, SW2, SW21, SW22, SW23, SW24, SW25, SW26, SW27, SW29, SW3, SW30, SW31, SW33, SW34, SW35, SW37, SW38, SW39, SW4, SW40, SW41, SW42, SW43, SW45, SW46, SW47, SW49, SW5, SW50, SW51, SW52, SW53, SW54, SW55, SW57, SW58, SW59, SW6, SW60, SW63, SW7, SW8, SW9: footprint Keebio-Parts:MX_PCB_100H -> footprints:100-minimal; symbol keyboard_parts:SW_PUSH -> rick-kicad-lib:switch
- SW18, SW20, SW28, SW64: footprint Keebio-Parts:MX_PCB_125H -> footprints:125-minimal; symbol keyboard_parts:SW_PUSH -> rick-kicad-lib:switch
- SW19, SW61: footprint Keebio-Parts:MX_PCB_175H -> footprints:175-minimal; symbol keyboard_parts:SW_PUSH -> rick-kicad-lib:switch
- SW32: footprint Keebio-Parts:MX_PCB_225H -> footprints:225-minimal; symbol keyboard_parts:SW_PUSH -> rick-kicad-lib:switch
- SW48: footprint Keebio-Parts:MX_PCB_275H -> footprints:275-minimal; symbol keyboard_parts:SW_PUSH -> rick-kicad-lib:switch
- SW62: footprint Keebio-Parts:MX_PCB_150H -> footprints:150-minimal; symbol keyboard_parts:SW_PUSH -> rick-kicad-lib:switch
- U1: footprint promicro:ProMicro -> footprints:promicro; symbol promicro:ProMicro -> rick-kicad-lib:promicro

Commit message: shorter.
Parts:
- SW19, SW61: footprint footprints:175-minimal -> footprints:150-minimal
- SW48: footprint footprints:275-minimal -> footprints:225-minimal
- SW52: footprint footprints:100-minimal -> footprints:125-minimal
- SW62: footprint footprints:150-minimal -> footprints:125-minimal
Changed lines of the file:
@@
 F 0 "SW62" H 13200 2055 50  0000 C CNN
 F 1 "SW_PUSH" H 13200 1964 50  0000 C CNN
-F 2 "footprints:150-minimal" H 13200 1800 60  0001 C CNN
+F 2 "footprints:125-minimal" H 13200 1800 60  0001 C CNN
 F 3 "" H 13200 1800 60  0000 C CNN
 	1    13200 1800
@@
 F 0 "SW61" H 13200 1305 50  0000 C CNN
 F 1 "SW_PUSH" H 13200 1214 50  0000 C CNN
-F 2 "footprints:175-minimal" H 13200 1050 60  0001 C CNN
+F 2 "footprints:150-minimal" H 13200 1050 60  0001 C CNN
 F 3 "" H 13200 1050 60  0000 C CNN
 	1    13200 1050
@@
 F 0 "SW48" H 10050 3955 50  0000 C CNN
 F 1 "SW_PUSH" H 10050 3864 50  0000 C CNN
-F 2 "footprints:275-minimal" H 10050 3700 60  0001 C CNN
+F 2 "footprints:225-minimal" H 10050 3700 60  0001 C CNN
 F 3 "" H 10050 3700 60  0000 C CNN
 	1    10050 3700
@@
 F 0 "SW19" H 4450 2955 50  0000 C CNN
 F 1 "SW_PUSH" H 4450 2864 50  0000 C CNN
-F 2 "footprints:175-minimal" H 4450 2700 60  0001 C CNN
+F 2 "footprints:150-minimal" H 4450 2700 60  0001 C CNN
 F 3 "" H 4450 2700 60  0000 C CNN
 	1    4450 2700
@@
 F 0 "SW52" H 10800 3955 50  0000 C CNN
 F 1 "SW_PUSH" H 10800 3864 50  0000 C CNN
-F 2 "footprints:100-minimal" H 10800 3700 60  0001 C CNN
+F 2 "footprints:125-minimal" H 10800 3700 60  0001 C CNN
 F 3 "" H 10800 3700 60  0000 C CNN
 	1    10800 3700
